File: ESP32-Seed-2.kicad_pcb (KiCad board)
At the start: 4 copper layers, 20 x 40.1 mm, 59 parts, among them J101 Conn_01x12_Pin, J102 Conn_01x12_Pin, J3 USB_C_Receptacle, SW1 SW_Push, SW2 SW_Push, U1 PCM5102, U101 W25Q128JVS, U102 PCM1808, U104 MC78L05_SOT89, U2 ESP32-S3, U3 AMS1117-3.3, Y1 40MHz

Commit message: Fixed Flash Chip Footprint
Parts:
- U101: footprint Package_SO:SOIC-8_3.9x4.9mm_P1.27mm -> Package_SO:SOIC-8_5.3x5.3mm_P1.27mm
- moved C15 0.73 mm to (164.7, 108.7)
- moved R8 0.69 mm to (166.2, 108.7)
- moved C4 0.52 mm to (165.3, 111.2)
- moved U101 0.36 mm to (159.3, 110.0)
- moved C3 0.28 mm to (161.4, 111.2)
- moved C108 0.24 mm to (163.0, 111.2)
- moved C105 0.20 mm to (159.9, 111.2)
- moved R7 0.08 mm to (161.7, 105.5)
- moved R11 0.08 mm to (156.9, 105.5)
- moved R10 0.08 mm to (158.5, 105.5)
- moved R6 0.08 mm to (160.1, 105.5)
Routing:
- net GND: track 114.2 -> 131.8 mm
- net +3V3: track 36.8 -> 41.2 mm, vias 15 -> 14
- net GPIO13: track 22.1 -> 24.9 mm
- net OUTL: track 16.3 -> 18.1 mm
- net OUTR: track 18.9 -> 17.6 mm
- net Net-(U101-~{HOLD}/~{RESET}/IO_{3}): track 8.30 -> 9.66 mm
- net Net-(U1-CAPP): track 5.74 -> 6.89 mm
- net Net-(U101-~{CS}): track 7.29 -> 6.39 mm
- net Net-(U1-CAPM): track 2.86 -> 3.64 mm
- net SPI_CS: track 19.4 -> 18.8 mm
- net Net-(U101-CLK): track 6.86 -> 7.49 mm
- net +5V: track 29.7 -> 30.3 mm
- net GPIO9: track 13.8 -> 13.2 mm
- net SPI_HD: track 24.2 -> 24.8 mm
- net Net-(U101-DI/IO_{0}): track 5.32 -> 4.73 mm
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Other:
- board size 20 x 40.1 mm -> 20 x 40.2 mm
- board text added: "VP2.0"
- board text removed: "VP1.0"
