File: ESP32-Seed-2.kicad_sch (KiCad schematic)
At the start: 59 parts, among them J101 Conn_01x12_Pin, J102 Conn_01x12_Pin, J3 USB_C_Receptacle, SW1 SW_Push, SW2 SW_Push, U1 PCM5102, U101 W25Q128JVS, U102 PCM1808, U104 MC78L05_SOT89, U2 ESP32-S3, U3 AMS1117-3.3, Y1 40MHz

Commit message: Fixed Flash Chip Footprint
Parts:
- U101: footprint Package_SO:SOIC-8_3.9x4.9mm_P1.27mm -> Package_SO:SOIC-8_5.3x5.3mm_P1.27mm
Changed lines of the file:
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@@
 			)
 		)
-		(property "Footprint" "Package_SO:SOIC-8_3.9x4.9mm_P1.27mm"
+		(property "Footprint" "Package_SO:SOIC-8_5.3x5.3mm_P1.27mm"
 			(at 213.36 46.99 0)
 			(effects
